File: hw/sch_pcb/_autosave-PCRD04B.kicad_pcb (KiCad board)
At the start: 2 copper layers, 60.5 x 40.1 mm, 62 parts, among them J1 3.6V, J11 HEADER_2x01_PARALLEL, J2 HEADER_2x01_PARALLEL, J3 HEADER_2x01_PARALLEL, J4 HEADER_2x01_PARALLEL, J5 HEADER_2x01_PARALLEL, J6 HEADER_2x01_PARALLEL, J7 HEADER_2x01_PARALLEL, M1 HOLE, M2 HOLE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

Commit message: 3D model
Parts:
- C2, C21, C22, C23, C24, C25: footprint Mlab_L:FIR1 -> Mlab_L:FIR_0805
