File: hw/sch_pcb/PCRD04B.kicad_sch (KiCad schematic)
At the start: 62 parts, among them J1 3.6V, J11 HEADER_2x01_PARALLEL, J2 HEADER_2x01_PARALLEL, J3 HEADER_2x01_PARALLEL, J4 HEADER_2x01_PARALLEL, J5 HEADER_2x01_PARALLEL, J6 HEADER_2x01_PARALLEL, J7 HEADER_2x01_PARALLEL, M1 HOLE, M2 HOLE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

Commit message: clean and update templates
Other:
- title: NAME -> (none)

Commit message: Update PCRD04B.kicad_sch
Other:
- company: Mlab www.mlab.cz -> MLAB www.mlab.cz
Changed lines of the file:
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@@
   (title_block
     (date "%F")
-    (company "Mlab www.mlab.cz")
+    (company "MLAB www.mlab.cz")
     (comment 1 "VERSION")
-    (comment 2 "Short description \\nTwo lines are maximum")
-    (comment 3 "nickname <email@example.com>")
-    (comment 4 "BSD")
+    (comment 2 "Battery biasedPIN diode\\ncosmic radiation detector")
+    (comment 3 "Martin Kakona <kakl@mlab.cz>")
+    (comment 4 "GPL 3")
   )
   (junction (at 93.98 153.67) (diameter 1.016) (color 0 0 0 0)
